Commit message: ✨feat:初期位置の指定

File: gazebo_simulator/urdf/swerve_bot.urdf.xacro (robot description, xacro)
@@ -6,5 +6,5 @@
   <!-- 初期位置の指定 -->
   <joint name="robot_footprint_joint" type="fixed">
-    <origin xyz="-5.5 0 0" rpy="0 0 0" />
+    <origin xyz="0 0 0" rpy="0 0 0" />
     <parent link="robot_footprint"/>
     <child link="chassis" />

Commit message: lidarのパラメータをUST-20LXに変更

File: gazebo_simulator/urdf/swerve_bot.urdf.xacro (robot description, xacro)
@@ -20,5 +20,5 @@
       <origin xyz="0 0 0" rpy=" 0 0 0"/>
       <geometry>
-        <box size=".8 .8 .1"/>
+        <box size=".8 .8 .15"/>
       </geometry>
     </collision>
@@ -26,5 +26,5 @@
       <origin xyz="0 0 0" rpy=" 0 0 0"/>
       <geometry>
-        <box size=".8 .8 .1"/>
+        <box size=".8 .8 .15"/>
       </geometry>
     </visual>
@@ -179,5 +179,5 @@
   </joint>
   <joint type="fixed" name="camera_joint">
-    <origin xyz="0.15 0 0.1" rpy="0 0 0"/>
+    <origin xyz="0.3 0 0.1" rpy="0 0 0"/>
     <child link="camera"/>
     <parent link="chassis"/>

Commit message: ✨feat:ステアのlidarを実機に合わせる

File: gazebo_simulator/urdf/swerve_bot.urdf.xacro (robot description, xacro)
@@ -142,5 +142,5 @@
       <origin xyz="0 0 0" rpy="0 0 0" />
       <geometry>
-        <box size="0.05 0.05 0.01"/>
+        <box size="0.05 0.05 0"/>
       </geometry>
     </collision>
@@ -185,5 +185,5 @@
   </joint>
   <joint type="fixed" name="hokuyo_joint">
-    <origin xyz="0.4 0 -0.07" rpy="0 0 0"/>
+    <origin xyz="0.425 0 -0.07" rpy="3.14159 0 0"/>
     <child link="hokuyo"/>
     <parent link="chassis"/>
