Commit message: RRのlidarを反転

File: gazebo_simulator/urdf/rr.urdf.xacro (robot description, xacro)
@@ -185,5 +185,5 @@
   <!-- 地面からセンサ:0.1711 - シャーシからタイヤ:0.05 + タイヤ半径:0.05 = 0.0711 -->
   <joint type="fixed" name="hokuyo_joint">
-    <origin xyz="0.1975 0 0.0711" rpy="0 0 0"/>
+    <origin xyz="0.1975 0 0.0711" rpy="3.14159 0 0"/>
     <child link="hokuyo"/>
     <parent link="chassis"/>
