Commit message: ✨feat:RRの追加

File: gazebo_simulator/urdf/er.urdf.xacro (robot description, xacro)
@@ -1,6 +1,6 @@
 <?xml version='1.0'?>
-<robot name="swerve_bot"
+<robot name="er"
   xmlns:xacro="http://www.ros.org/wiki/xacro">
-  <xacro:include filename="swerve_bot.gazebo" />
+  <xacro:include filename="sensors.gazebo" />
   <link name="robot_footprint"></link>
   <!-- 初期位置の指定 -->
@@ -11,5 +11,4 @@
   </joint>
   <link name='chassis'>
-    <pose>0 0 0.1 0 0 0</pose>
     <inertial>
       <mass value="15.0"/>
@@ -134,5 +133,5 @@
       <origin xyz="0 0 0" rpy="0 0 0" />
       <geometry>
-        <!-- <mesh filename="$(find swerve_bot)/meshes/hokuyo.dae"/> -->
+        <!-- <mesh filename="$(find er)/meshes/hokuyo.dae"/> -->
         <box size="0.05 0.05 0.05"/>
       </geometry>

Commit message: first commit

File: gazebo_simulator/urdf/er.urdf.xacro (robot description, xacro)
@@ -19,5 +19,5 @@
       <origin xyz="0 0 0" rpy=" 0 0 0"/>
       <geometry>
-        <box size=".8 .8 .15"/>
+        <box size=".5 .5 .15"/>
       </geometry>
     </collision>
@@ -25,5 +25,5 @@
       <origin xyz="0 0 0" rpy=" 0 0 0"/>
       <geometry>
-        <box size=".8 .8 .15"/>
+        <box size=".5 .5 .15"/>
       </geometry>
     </visual>
@@ -38,11 +38,11 @@
       <origin xyz="0.0 0 0" rpy=" 0 1.5707 1.5707"/>
       <geometry>
-        <cylinder length="0.05" radius="0.1"/>
-      </geometry>
-    </visual>
-    <collision>
-      <origin xyz="0.0 0 0" rpy=" 0 1.5707 1.5707"/>
-      <geometry>
-        <cylinder length="0.05" radius="0.1"/>
+        <cylinder length="0.05" radius="0.05"/>
+      </geometry>
+    </visual>
+    <collision>
+      <origin xyz="0.0 0 0" rpy=" 0 1.5707 1.5707"/>
+      <geometry>
+        <cylinder length="0.05" radius="0.05"/>
       </geometry>
     </collision>
@@ -57,11 +57,11 @@
       <origin xyz="0.0 0 0" rpy=" 0 1.5707 1.5707"/>
       <geometry>
-        <cylinder length="0.05" radius="0.1"/>
-      </geometry>
-    </visual>
-    <collision>
-      <origin xyz="0.0 0 0" rpy=" 0 1.5707 1.5707"/>
-      <geometry>
-        <cylinder length="0.05" radius="0.1"/>
+        <cylinder length="0.05" radius="0.05"/>
+      </geometry>
+    </visual>
+    <collision>
+      <origin xyz="0.0 0 0" rpy=" 0 1.5707 1.5707"/>
+      <geometry>
+        <cylinder length="0.05" radius="0.05"/>
       </geometry>
     </collision>
@@ -76,11 +76,11 @@
       <origin xyz="0.0 0 0" rpy=" 0 1.5707 1.5707"/>
       <geometry>
-        <cylinder length="0.05" radius="0.1"/>
-      </geometry>
-    </visual>
-    <collision>
-      <origin xyz="0.0 0 0" rpy=" 0 1.5707 1.5707"/>
-      <geometry>
-        <cylinder length="0.05" radius="0.1"/>
+        <cylinder length="0.05" radius="0.05"/>
+      </geometry>
+    </visual>
+    <collision>
+      <origin xyz="0.0 0 0" rpy=" 0 1.5707 1.5707"/>
+      <geometry>
+        <cylinder length="0.05" radius="0.05"/>
       </geometry>
     </collision>
@@ -95,11 +95,11 @@
       <origin xyz="0.0 0 0" rpy=" 0 1.5707 1.5707"/>
       <geometry>
-        <cylinder length="0.05" radius="0.1"/>
-      </geometry>
-    </visual>
-    <collision>
-      <origin xyz="0.0 0 0" rpy=" 0 1.5707 1.5707"/>
-      <geometry>
-        <cylinder length="0.05" radius="0.1"/>
+        <cylinder length="0.05" radius="0.05"/>
+      </geometry>
+    </visual>
+    <collision>
+      <origin xyz="0.0 0 0" rpy=" 0 1.5707 1.5707"/>
+      <geometry>
+        <cylinder length="0.05" radius="0.05"/>
       </geometry>
     </collision>

Commit message: map変更

File: gazebo_simulator/urdf/er.urdf.xacro (robot description, xacro)
@@ -19,5 +19,5 @@
       <origin xyz="0 0 0" rpy=" 0 0 0"/>
       <geometry>
-        <box size=".5 .5 .15"/>
+        <box size=".5 .5 .65"/>
       </geometry>
     </collision>
@@ -25,5 +25,5 @@
       <origin xyz="0 0 0" rpy=" 0 0 0"/>
       <geometry>
-        <box size=".5 .5 .15"/>
+        <box size=".5 .5 .7"/>
       </geometry>
     </visual>
@@ -146,5 +146,5 @@
   </link>
   <joint type="continuous" name="front_left_wheel_joint">
-    <origin xyz="0.3 0.3 0" rpy="0 0 -0.7853"/>
+    <origin xyz="0.2 0.2 -0.35" rpy="0 0 -0.7853"/>
     <child link="front_left_wheel"/>
     <parent link="chassis"/>
@@ -154,5 +154,5 @@
   </joint>
   <joint type="continuous" name="front_right_wheel_joint">
-    <origin xyz="0.3 -0.3 0" rpy="0 0 0.7853"/>
+    <origin xyz="0.22 -0.22 -0.35" rpy="0 0 0.7853"/>
     <child link="front_right_wheel"/>
     <parent link="chassis"/>
@@ -162,5 +162,5 @@
   </joint>
   <joint type="continuous" name="back_left_wheel_joint">
-    <origin xyz="-0.3 0.3 0" rpy="0 0 3.9269"/>
+    <origin xyz="-0.22 0.22 -0.35" rpy="0 0 3.9269"/>
     <child link="back_left_wheel"/>
     <parent link="chassis"/>
@@ -170,5 +170,5 @@
   </joint>
   <joint type="continuous" name="back_right_wheel_joint">
-    <origin xyz="-0.3 -0.3 0" rpy="0 0 -3.9269"/>
+    <origin xyz="-0.22 -0.22 -0.35" rpy="0 0 -3.9269"/>
     <child link="back_right_wheel"/>
     <parent link="chassis"/>
@@ -178,5 +178,5 @@
   </joint>
   <joint type="fixed" name="camera_joint">
-    <origin xyz="0.3 0 0.1" rpy="0 0 0"/>
+    <origin xyz="0.3 0 -0.25" rpy="0 0 0"/>
     <child link="camera"/>
     <parent link="chassis"/>
@@ -184,5 +184,5 @@
   </joint>
   <joint type="fixed" name="hokuyo_joint">
-    <origin xyz="0.425 0 -0.07" rpy="3.14159 0 0"/>
+    <origin xyz="0.3 0 -0.35" rpy="3.14159 0 0"/>
     <child link="hokuyo"/>
     <parent link="chassis"/>

File: gazebo_simulator/urdf/rr.urdf.xacro (robot description, xacro)
@@ -19,5 +19,5 @@
       <origin xyz="0 0 0" rpy=" 0 0 0"/>
       <geometry>
-        <box size=".46 .46 .15"/>
+        <box size=".5 .5 .7"/>
       </geometry>
     </collision>
@@ -25,5 +25,5 @@
       <origin xyz="0 0 0" rpy=" 0 0 0"/>
       <geometry>
-        <box size=".46 .46 .15"/>
+        <box size=".5 .5 .7"/>
       </geometry>
     </visual>
@@ -146,5 +146,5 @@
   </link>
   <joint type="continuous" name="front_left_wheel_joint">
-    <origin xyz="0.15 0.15 -0.05" rpy="0 0 -0.7853"/>
+    <origin xyz="0.3 0.3 0" rpy="0 0 -0.7853"/>
     <child link="front_left_wheel"/>
     <parent link="chassis"/>
@@ -154,5 +154,5 @@
   </joint>
   <joint type="continuous" name="front_right_wheel_joint">
-    <origin xyz="0.15 -0.15 -0.05" rpy="0 0 0.7853"/>
+    <origin xyz="0.3 -0.3 0" rpy="0 0 0.7853"/>
     <child link="front_right_wheel"/>
     <parent link="chassis"/>
@@ -162,5 +162,5 @@
   </joint>
   <joint type="continuous" name="back_left_wheel_joint">
-    <origin xyz="-0.15 0.15 -0.05" rpy="0 0 3.9269"/>
+    <origin xyz="-0.3 0.3 0" rpy="0 0 3.9269"/>
     <child link="back_left_wheel"/>
     <parent link="chassis"/>
@@ -170,5 +170,5 @@
   </joint>
   <joint type="continuous" name="back_right_wheel_joint">
-    <origin xyz="-0.15 -0.15 -0.05" rpy="0 0 -3.9269"/>
+    <origin xyz="-0.3 -0.3 0" rpy="0 0 -3.9269"/>
     <child link="back_right_wheel"/>
     <parent link="chassis"/>
@@ -178,12 +178,11 @@
   </joint>
   <joint type="fixed" name="camera_joint">
-    <origin xyz="0.1 0 0.1" rpy="0 0 0"/>
+    <origin xyz="0.3 0 0.1" rpy="0 0 0"/>
     <child link="camera"/>
     <parent link="chassis"/>
     <axis xyz="0 1 0" rpy="0 0 0"/>
   </joint>
-  <!-- 地面からセンサ:0.1711 - シャーシからタイヤ:0.05 + タイヤ半径:0.05 = 0.0711 -->
   <joint type="fixed" name="hokuyo_joint">
-    <origin xyz="0.1975 0 0.0711" rpy="3.14159 0 0"/>
+    <origin xyz="0.425 0 -0.07" rpy="3.14159 0 0"/>
     <child link="hokuyo"/>
     <parent link="chassis"/>

Commit message: 坂バグ修正

File: gazebo_simulator/urdf/er.urdf.xacro (robot description, xacro)
@@ -25,5 +25,5 @@
       <origin xyz="0 0 0" rpy=" 0 0 0"/>
       <geometry>
-        <box size=".5 .5 .7"/>
+        <box size=".5 .5 .65"/>
       </geometry>
     </visual>
@@ -178,5 +178,5 @@
   </joint>
   <joint type="fixed" name="camera_joint">
-    <origin xyz="0.3 0 -0.25" rpy="0 0 0"/>
+    <origin xyz="0.3 0 -0.35" rpy="0 0 0"/>
     <child link="camera"/>
     <parent link="chassis"/>
@@ -184,5 +184,5 @@
   </joint>
   <joint type="fixed" name="hokuyo_joint">
-    <origin xyz="0.3 0 -0.35" rpy="3.14159 0 0"/>
+    <origin xyz="0.3 0 -0.25" rpy="3.14159 0 0"/>
     <child link="hokuyo"/>
     <parent link="chassis"/>

File: gazebo_simulator/urdf/rr.urdf.xacro (robot description, xacro)
@@ -19,5 +19,5 @@
       <origin xyz="0 0 0" rpy=" 0 0 0"/>
       <geometry>
-        <box size=".5 .5 .7"/>
+        <box size=".5 .5 .65"/>
       </geometry>
     </collision>
@@ -25,5 +25,5 @@
       <origin xyz="0 0 0" rpy=" 0 0 0"/>
       <geometry>
-        <box size=".5 .5 .7"/>
+        <box size=".5 .5 .65"/>
       </geometry>
     </visual>
@@ -146,5 +146,5 @@
   </link>
   <joint type="continuous" name="front_left_wheel_joint">
-    <origin xyz="0.3 0.3 0" rpy="0 0 -0.7853"/>
+    <origin xyz="0.2 0.2 -0.35" rpy="0 0 -0.7853"/>
     <child link="front_left_wheel"/>
     <parent link="chassis"/>
@@ -154,5 +154,5 @@
   </joint>
   <joint type="continuous" name="front_right_wheel_joint">
-    <origin xyz="0.3 -0.3 0" rpy="0 0 0.7853"/>
+    <origin xyz="0.22 -0.22 -0.35" rpy="0 0 0.7853"/>
     <child link="front_right_wheel"/>
     <parent link="chassis"/>
@@ -162,5 +162,5 @@
   </joint>
   <joint type="continuous" name="back_left_wheel_joint">
-    <origin xyz="-0.3 0.3 0" rpy="0 0 3.9269"/>
+    <origin xyz="-0.22 0.22 -0.35" rpy="0 0 3.9269"/>
     <child link="back_left_wheel"/>
     <parent link="chassis"/>
@@ -170,5 +170,5 @@
   </joint>
   <joint type="continuous" name="back_right_wheel_joint">
-    <origin xyz="-0.3 -0.3 0" rpy="0 0 -3.9269"/>
+    <origin xyz="-0.22 -0.22 -0.35" rpy="0 0 -3.9269"/>
     <child link="back_right_wheel"/>
     <parent link="chassis"/>
@@ -178,5 +178,5 @@
   </joint>
   <joint type="fixed" name="camera_joint">
-    <origin xyz="0.3 0 0.1" rpy="0 0 0"/>
+    <origin xyz="0.3 0 -0.25" rpy="0 0 0"/>
     <child link="camera"/>
     <parent link="chassis"/>
@@ -184,5 +184,5 @@
   </joint>
   <joint type="fixed" name="hokuyo_joint">
-    <origin xyz="0.425 0 -0.07" rpy="3.14159 0 0"/>
+    <origin xyz="0.3 0 -0.35" rpy="3.14159 0 0"/>
     <child link="hokuyo"/>
     <parent link="chassis"/>

Commit message: gazebo修正

File: gazebo_simulator/urdf/er.urdf.xacro (robot description, xacro)
@@ -1,4 +1,4 @@
 <?xml version='1.0'?>
-<robot name="er"
+<robot name="rr"
   xmlns:xacro="http://www.ros.org/wiki/xacro">
   <xacro:include filename="sensors.gazebo" />
@@ -178,5 +178,5 @@
   </joint>
   <joint type="fixed" name="camera_joint">
-    <origin xyz="0.3 0 -0.35" rpy="0 0 0"/>
+    <origin xyz="0.3 0 -0.25" rpy="0 0 0"/>
     <child link="camera"/>
     <parent link="chassis"/>
@@ -184,5 +184,5 @@
   </joint>
   <joint type="fixed" name="hokuyo_joint">
-    <origin xyz="0.3 0 -0.25" rpy="3.14159 0 0"/>
+    <origin xyz="0.3 0 -0.35" rpy="3.14159 0 0"/>
     <child link="hokuyo"/>
     <parent link="chassis"/>

Commit message: node_list,edge_list追加

File: gazebo_simulator/urdf/er.urdf.xacro (robot description, xacro)
@@ -19,5 +19,5 @@
       <origin xyz="0 0 0" rpy=" 0 0 0"/>
       <geometry>
-        <box size=".5 .5 .15"/>
+        <box size=".5 .5 .65"/>
       </geometry>
     </collision>
@@ -25,5 +25,5 @@
       <origin xyz="0 0 0" rpy=" 0 0 0"/>
       <geometry>
-        <box size=".5 .5 .15"/>
+        <box size=".5 .5 .65"/>
       </geometry>
     </visual>
@@ -146,5 +146,5 @@
   </link>
   <joint type="continuous" name="front_left_wheel_joint">
-    <origin xyz="0.3 0.3 0" rpy="0 0 -0.7853"/>
+    <origin xyz="0.2 0.2 -0.35" rpy="0 0 -0.7853"/>
     <child link="front_left_wheel"/>
     <parent link="chassis"/>
@@ -154,5 +154,5 @@
   </joint>
   <joint type="continuous" name="front_right_wheel_joint">
-    <origin xyz="0.3 -0.3 0" rpy="0 0 0.7853"/>
+    <origin xyz="0.22 -0.22 -0.35" rpy="0 0 0.7853"/>
     <child link="front_right_wheel"/>
     <parent link="chassis"/>
@@ -162,5 +162,5 @@
   </joint>
   <joint type="continuous" name="back_left_wheel_joint">
-    <origin xyz="-0.3 0.3 0" rpy="0 0 3.9269"/>
+    <origin xyz="-0.22 0.22 -0.35" rpy="0 0 3.9269"/>
     <child link="back_left_wheel"/>
     <parent link="chassis"/>
@@ -170,5 +170,5 @@
   </joint>
   <joint type="continuous" name="back_right_wheel_joint">
-    <origin xyz="-0.3 -0.3 0" rpy="0 0 -3.9269"/>
+    <origin xyz="-0.22 -0.22 -0.35" rpy="0 0 -3.9269"/>
     <child link="back_right_wheel"/>
     <parent link="chassis"/>
@@ -178,5 +178,5 @@
   </joint>
   <joint type="fixed" name="camera_joint">
-    <origin xyz="0.3 0 0.1" rpy="0 0 0"/>
+    <origin xyz="0.3 0 -0.25" rpy="0 0 0"/>
     <child link="camera"/>
     <parent link="chassis"/>
@@ -184,5 +184,5 @@
   </joint>
   <joint type="fixed" name="hokuyo_joint">
-    <origin xyz="0.425 0 -0.07" rpy="3.14159 0 0"/>
+    <origin xyz="0.3 0 -0.35" rpy="3.14159 0 0"/>
     <child link="hokuyo"/>
     <parent link="chassis"/>

Commit message: コート情報反映

File: gazebo_simulator/urdf/er.urdf.xacro (robot description, xacro)
@@ -154,5 +154,5 @@
   </joint>
   <joint type="continuous" name="front_right_wheel_joint">
-    <origin xyz="0.22 -0.22 -0.35" rpy="0 0 0.7853"/>
+    <origin xyz="0.2 -0.2 -0.35" rpy="0 0 0.7853"/>
     <child link="front_right_wheel"/>
     <parent link="chassis"/>
@@ -162,5 +162,5 @@
   </joint>
   <joint type="continuous" name="back_left_wheel_joint">
-    <origin xyz="-0.22 0.22 -0.35" rpy="0 0 3.9269"/>
+    <origin xyz="-0.2 0.2 -0.35" rpy="0 0 3.9269"/>
     <child link="back_left_wheel"/>
     <parent link="chassis"/>
@@ -170,5 +170,5 @@
   </joint>
   <joint type="continuous" name="back_right_wheel_joint">
-    <origin xyz="-0.22 -0.22 -0.35" rpy="0 0 -3.9269"/>
+    <origin xyz="-0.2 -0.2 -0.35" rpy="0 0 -3.9269"/>
     <child link="back_right_wheel"/>
     <parent link="chassis"/>

File: gazebo_simulator/urdf/rr.urdf.xacro (robot description, xacro)
@@ -1,4 +1,4 @@
 <?xml version='1.0'?>
-<robot name="rr"
+<robot name="er"
   xmlns:xacro="http://www.ros.org/wiki/xacro">
   <xacro:include filename="sensors.gazebo" />
@@ -154,5 +154,5 @@
   </joint>
   <joint type="continuous" name="front_right_wheel_joint">
-    <origin xyz="0.22 -0.22 -0.35" rpy="0 0 0.7853"/>
+    <origin xyz="0.2 -0.2 -0.35" rpy="0 0 0.7853"/>
     <child link="front_right_wheel"/>
     <parent link="chassis"/>
@@ -162,5 +162,5 @@
   </joint>
   <joint type="continuous" name="back_left_wheel_joint">
-    <origin xyz="-0.22 0.22 -0.35" rpy="0 0 3.9269"/>
+    <origin xyz="-0.2 0.2 -0.35" rpy="0 0 3.9269"/>
     <child link="back_left_wheel"/>
     <parent link="chassis"/>
@@ -170,5 +170,5 @@
   </joint>
   <joint type="continuous" name="back_right_wheel_joint">
-    <origin xyz="-0.22 -0.22 -0.35" rpy="0 0 -3.9269"/>
+    <origin xyz="-0.2 -0.2 -0.35" rpy="0 0 -3.9269"/>
     <child link="back_right_wheel"/>
     <parent link="chassis"/>

Commit message: gazebo改善

File: gazebo_simulator/urdf/er.urdf.xacro (robot description, xacro)
@@ -1,4 +1,4 @@
 <?xml version='1.0'?>
-<robot name="rr"
+<robot name="er"
   xmlns:xacro="http://www.ros.org/wiki/xacro">
   <xacro:include filename="sensors.gazebo" />
@@ -19,5 +19,5 @@
       <origin xyz="0 0 0" rpy=" 0 0 0"/>
       <geometry>
-        <box size=".5 .5 .65"/>
+        <box size=".5 .5 .5"/>
       </geometry>
     </collision>
@@ -25,5 +25,5 @@
       <origin xyz="0 0 0" rpy=" 0 0 0"/>
       <geometry>
-        <box size=".5 .5 .65"/>
+        <box size=".5 .5 .5"/>
       </geometry>
     </visual>
@@ -38,11 +38,11 @@
       <origin xyz="0.0 0 0" rpy=" 0 1.5707 1.5707"/>
       <geometry>
-        <cylinder length="0.05" radius="0.05"/>
-      </geometry>
-    </visual>
-    <collision>
-      <origin xyz="0.0 0 0" rpy=" 0 1.5707 1.5707"/>
-      <geometry>
-        <cylinder length="0.05" radius="0.05"/>
+        <cylinder length="0.05" radius="0.07"/>
+      </geometry>
+    </visual>
+    <collision>
+      <origin xyz="0.0 0 0" rpy=" 0 1.5707 1.5707"/>
+      <geometry>
+        <cylinder length="0.05" radius="0.07"/>
       </geometry>
     </collision>
@@ -57,11 +57,11 @@
       <origin xyz="0.0 0 0" rpy=" 0 1.5707 1.5707"/>
       <geometry>
-        <cylinder length="0.05" radius="0.05"/>
-      </geometry>
-    </visual>
-    <collision>
-      <origin xyz="0.0 0 0" rpy=" 0 1.5707 1.5707"/>
-      <geometry>
-        <cylinder length="0.05" radius="0.05"/>
+        <cylinder length="0.05" radius="0.07"/>
+      </geometry>
+    </visual>
+    <collision>
+      <origin xyz="0.0 0 0" rpy=" 0 1.5707 1.5707"/>
+      <geometry>
+        <cylinder length="0.05" radius="0.07"/>
       </geometry>
     </collision>
@@ -76,11 +76,11 @@
       <origin xyz="0.0 0 0" rpy=" 0 1.5707 1.5707"/>
       <geometry>
-        <cylinder length="0.05" radius="0.05"/>
-      </geometry>
-    </visual>
-    <collision>
-      <origin xyz="0.0 0 0" rpy=" 0 1.5707 1.5707"/>
-      <geometry>
-        <cylinder length="0.05" radius="0.05"/>
+        <cylinder length="0.05" radius="0.07"/>
+      </geometry>
+    </visual>
+    <collision>
+      <origin xyz="0.0 0 0" rpy=" 0 1.5707 1.5707"/>
+      <geometry>
+        <cylinder length="0.05" radius="0.07"/>
       </geometry>
     </collision>
@@ -95,11 +95,11 @@
       <origin xyz="0.0 0 0" rpy=" 0 1.5707 1.5707"/>
       <geometry>
-        <cylinder length="0.05" radius="0.05"/>
-      </geometry>
-    </visual>
-    <collision>
-      <origin xyz="0.0 0 0" rpy=" 0 1.5707 1.5707"/>
-      <geometry>
-        <cylinder length="0.05" radius="0.05"/>
+        <cylinder length="0.05" radius="0.07"/>
+      </geometry>
+    </visual>
+    <collision>
+      <origin xyz="0.0 0 0" rpy=" 0 1.5707 1.5707"/>
+      <geometry>
+        <cylinder length="0.05" radius="0.07"/>
       </geometry>
     </collision>
@@ -146,5 +146,5 @@
   </link>
   <joint type="continuous" name="front_left_wheel_joint">
-    <origin xyz="0.2 0.2 -0.35" rpy="0 0 -0.7853"/>
+    <origin xyz="0.2 0.2 -0.3" rpy="0 0 -0.7853"/>
     <child link="front_left_wheel"/>
     <parent link="chassis"/>
@@ -154,5 +154,5 @@
   </joint>
   <joint type="continuous" name="front_right_wheel_joint">
-    <origin xyz="0.2 -0.2 -0.35" rpy="0 0 0.7853"/>
+    <origin xyz="0.2 -0.2 -0.3" rpy="0 0 0.7853"/>
     <child link="front_right_wheel"/>
     <parent link="chassis"/>
@@ -162,5 +162,5 @@
   </joint>
   <joint type="continuous" name="back_left_wheel_joint">
-    <origin xyz="-0.2 0.2 -0.35" rpy="0 0 3.9269"/>
+    <origin xyz="-0.2 0.2 -0.3" rpy="0 0 3.9269"/>
     <child link="back_left_wheel"/>
     <parent link="chassis"/>
@@ -170,5 +170,5 @@
   </joint>
   <joint type="continuous" name="back_right_wheel_joint">
-    <origin xyz="-0.2 -0.2 -0.35" rpy="0 0 -3.9269"/>
+    <origin xyz="-0.2 -0.2 -0.3" rpy="0 0 -3.9269"/>
     <child link="back_right_wheel"/>
     <parent link="chassis"/>
@@ -178,5 +178,5 @@
   </joint>
   <joint type="fixed" name="camera_joint">
-    <origin xyz="0.3 0 -0.25" rpy="0 0 0"/>
+    <origin xyz="0.3 0 0.1" rpy="0 0 0"/>
     <child link="camera"/>
     <parent link="chassis"/>
@@ -184,5 +184,5 @@
   </joint>
   <joint type="fixed" name="hokuyo_joint">
-    <origin xyz="0.3 0 -0.35" rpy="3.14159 0 0"/>
+    <origin xyz="0.23 0 -0.33" rpy="3.14159 0 0"/>
     <child link="hokuyo"/>
     <parent link="chassis"/>

File: gazebo_simulator/urdf/rr.urdf.xacro (robot description, xacro)
@@ -1,4 +1,4 @@
 <?xml version='1.0'?>
-<robot name="er"
+<robot name="rr"
   xmlns:xacro="http://www.ros.org/wiki/xacro">
   <xacro:include filename="sensors.gazebo" />
